Commit message: single stair 0-1

File: wheelleg_description/urdf/Segway.xacro (robot description, xacro)
@@ -34,5 +34,5 @@
   </gazebo>
   <joint name="z_dof" type="prismatic">
-    <origin xyz="0 0 0" rpy="0 0 3.1415926"/>
+    <origin xyz="0 0 0" rpy="0 0 0"/>
     <parent link="static_base"/>
     <child link="z_dummy_link"/>
