Commit message: added plugin

File: wheelleg_description/urdf/Hexapod.xacro (robot description, xacro)
@@ -25,3 +25,9 @@
   <xacro:wheelLegJointConfig name="RM" />
   <xacro:wheelLegJointConfig name="RB" />
+  <xacro:WheelLegCollisionPluginConfig name="LF"/>
+  <xacro:WheelLegCollisionPluginConfig name="LM"/>
+  <xacro:WheelLegCollisionPluginConfig name="LB"/>
+  <xacro:WheelLegCollisionPluginConfig name="RF"/>
+  <xacro:WheelLegCollisionPluginConfig name="RM"/>
+  <xacro:WheelLegCollisionPluginConfig name="RB"/>
 </robot>

File: wheelleg_description/urdf/WheelLeg.xacro (robot description, xacro)
@@ -158,5 +158,5 @@
         </material>
       </visual>
-      <collision>
+      <collision name = "${name}RB_collision">
         <origin
           xyz="0 0 0"
@@ -264,5 +264,5 @@
         </material>
       </visual>
-      <collision>
+      <collision name = "${name}RA_collision">
         <origin
           xyz="0 0 0"

Commit message: added pose constraint for segway simulation

File: wheelleg_description/urdf/Hexapod.xacro (robot description, xacro)
@@ -11,11 +11,34 @@
     </plugin>
   </gazebo>
+    <!--define robot base link-->
+  <link name="base_link">
+    <inertial>
+      <origin xyz="0.05 0.05 0.05" rpy="0 0 0"/>
+      <mass value="1"/>
+      <inertia ixx="0.00167"  ixy="0"  ixz="0" iyy="0.00167" iyz="0" izz="0.00167" />
+    </inertial>
+    <visual>
+      <origin xyz="0 0 0" rpy="0 0 0" />
+      <geometry>
+        <box size="0.1 0.1 0.1" />
+      </geometry>
+      <material name="Cyan">
+        <color rgba="0 1.0 1.0 1.0"/>
+      </material>
+    </visual>
+    <!-- <collision>
+      <origin xyz="0 0 0" rpy="0 0 0"/>
+      <geometry>
+        <box size="0.1 0.1 0.1" />
+      </geometry>
+    </collision> -->
+  </link>
   <!--define joints-->
-  <xacro:LeftWheelLeg name="LF" x="0.4" y="0.2" z="0.02" />
-  <xacro:LeftWheelLeg name="LM" x="0" y="0.3" z="0.02" />
-  <xacro:LeftWheelLeg name="LB" x="-0.4" y="0.2" z="0.02" />
-  <xacro:RightWheelLeg name="RF" x="0.4" y="-0.2" z="0.02" />
-  <xacro:RightWheelLeg name="RM" x="0" y="-0.3" z="0.02" />
-  <xacro:RightWheelLeg name="RB" x="-0.4" y="-0.2" z="0.02" />
+  <xacro:LeftWheelLeg name="LF" x="0.4" y="0.2" z="0.02" parent="base_link"/>
+  <xacro:LeftWheelLeg name="LM" x="0" y="0.3" z="0.02" parent="base_link"/>
+  <xacro:LeftWheelLeg name="LB" x="-0.4" y="0.2" z="0.02" parent="base_link"/>
+  <xacro:RightWheelLeg name="RF" x="0.4" y="-0.2" z="0.02" parent="base_link"/>
+  <xacro:RightWheelLeg name="RM" x="0" y="-0.3" z="0.02" parent="base_link"/>
+  <xacro:RightWheelLeg name="RB" x="-0.4" y="-0.2" z="0.02" parent="base_link"/>
   <!--add gazebo joint configures-->
   <xacro:wheelLegJointConfig name="LF" />

File: wheelleg_description/urdf/Quadraped.xacro (robot description, xacro)
@@ -11,9 +11,32 @@
     </plugin>
   </gazebo>
+   <!--define robot base link-->
+  <link name="base_link">
+    <inertial>
+      <origin xyz="0.05 0.05 0.05" rpy="0 0 0"/>
+      <mass value="1"/>
+      <inertia ixx="0.00167"  ixy="0"  ixz="0" iyy="0.00167" iyz="0" izz="0.00167" />
+    </inertial>
+    <visual>
+      <origin xyz="0 0 0" rpy="0 0 0" />
+      <geometry>
+        <box size="0.1 0.1 0.1" />
+      </geometry>
+      <material name="Cyan">
+        <color rgba="0 1.0 1.0 1.0"/>
+      </material>
+    </visual>
+    <!-- <collision>
+      <origin xyz="0 0 0" rpy="0 0 0"/>
+      <geometry>
+        <box size="0.1 0.1 0.1" />
+      </geometry>
+    </collision> -->
+  </link>
   <!--define joints-->
-  <xacro:LeftWheelLeg name="LF" x="0.4" y="0.2" z="0.02" />
-  <xacro:LeftWheelLeg name="LB" x="-0.4" y="0.2" z="0.02" />
-  <xacro:RightWheelLeg name="RF" x="0.4" y="-0.2" z="0.02" />
-  <xacro:RightWheelLeg name="RB" x="-0.4" y="-0.2" z="0.02" />
+  <xacro:LeftWheelLeg name="LF" x="0.4" y="0.2" z="0.02" parent="base_link" />
+  <xacro:LeftWheelLeg name="LB" x="-0.4" y="0.2" z="0.02" parent="base_link"/>
+  <xacro:RightWheelLeg name="RF" x="0.4" y="-0.2" z="0.02" parent="base_link"/>
+  <xacro:RightWheelLeg name="RB" x="-0.4" y="-0.2" z="0.02" parent="base_link"/>
   <!--add gazebo joint configures-->
   <xacro:wheelLegJointConfig name="LF" />

File: wheelleg_description/urdf/Segway.xacro (robot description, xacro)
@@ -11,7 +11,82 @@
     </plugin>
   </gazebo>
+  <link name="static_base">
+    <inertial>
+      <origin xyz="0.05 0.05 0.05" rpy="0 0 0"/>
+      <mass value="1"/>
+      <inertia ixx="0.00167"  ixy="0"  ixz="0" iyy="0.00167" iyz="0" izz="0.00167" />
+    </inertial>
+    <visual>
+      <origin xyz="0 0 0" rpy="0 0 0" />
+      <geometry>
+        <box size="0.1 0.1 0.1" />
+      </geometry>
+      <material name="Cyan">
+        <color rgba="0 1.0 1.0 1.0"/>
+      </material>
+    </visual>
+  </link>
+  <gazebo>
+      <joint name ="weld" type="fixed">
+          <parent>world</parent>
+          <child>static_base</child>
+      </joint>
+  </gazebo>
+  <joint name="z_dof" type="prismatic">
+    <origin xyz="0 0 0" rpy="0 0 0"/>
+    <parent link="static_base"/>
+    <child link="z_dummy_link"/>
+    <limit effort="30" velocity="100.0" lower="-200" upper="200" />
+    <axis xyz="0 0 1"/>\
+  </joint>
+  <link name="z_dummy_link">
+    <inertial>
+      <origin xyz="0.05 0.05 0.05" rpy="0 0 0"/>
+      <mass value="1"/>
+      <inertia ixx="0.00167"  ixy="0"  ixz="0" iyy="0.00167" iyz="0" izz="0.00167" />
+    </inertial>
+    <visual>
+      <origin xyz="0 0 0" rpy="0 0 0" />
+      <geometry>
+        <box size="0.1 0.1 0.1" />
+      </geometry>
+      <material name="Cyan">
+        <color rgba="0 1.0 1.0 1.0"/>
+      </material>
+    </visual>
+  </link>
+  <joint name="x_dof" type="prismatic">
+    <origin xyz="0 0 0" rpy="0 0 0"/>
+    <parent link="z_dummy_link"/>
+    <child link="base_link"/>
+    <limit effort="30" velocity="100.0" lower="-200" upper="200" />
+    <axis xyz="1 0 0"/>\
+  </joint>
+  <!--define robot base link-->
+  <link name="base_link">
+    <inertial>
+      <origin xyz="0.05 0.05 0.05" rpy="0 0 0"/>
+      <mass value="1"/>
+      <inertia ixx="0.00167"  ixy="0"  ixz="0" iyy="0.00167" iyz="0" izz="0.00167" />
+    </inertial>
+    <visual>
+      <origin xyz="0 0 0" rpy="0 0 0" />
+      <geometry>
+        <box size="0.1 0.1 0.1" />
+      </geometry>
+      <material name="Cyan">
+        <color rgba="0 1.0 1.0 1.0"/>
+      </material>
+    </visual>
+    <!-- <collision>
+      <origin xyz="0 0 0" rpy="0 0 0"/>
+      <geometry>
+        <box size="0.1 0.1 0.1" />
+      </geometry>
+    </collision> -->
+  </link>
   <!--define joints-->
-  <xacro:LeftWheelLeg name="L" x="0" y="0.2" z="0.0" />
-  <xacro:RightWheelLeg name="R" x="0" y="-0.2" z="0.0" />
+  <xacro:LeftWheelLeg name="L" x="0" y="0.2" z="0.0" parent="base_link"/>
+  <xacro:RightWheelLeg name="R" x="0" y="-0.2" z="0.0" parent="base_link"/>
   <!--add gazebo joint configures-->
   <xacro:wheelLegJointConfig name="L" />

File: wheelleg_description/urdf/WheelLeg.xacro (robot description, xacro)
@@ -1,29 +1,6 @@
 <?xml version="1.0" encoding="utf-8"?>
 <robot xmlns:xacro="http://www.ros.org/wiki/xacro" >
-  <!--define robot base link-->
-  <link name="base_link">
-    <inertial>
-      <origin xyz="0.05 0.05 0.05" rpy="0 0 0"/>
-      <mass value="1"/>
-      <inertia ixx="0.00167"  ixy="0"  ixz="0" iyy="0.00167" iyz="0" izz="0.00167" />
-    </inertial>
-    <visual>
-      <origin xyz="0 0 0" rpy="0 0 0" />
-      <geometry>
-        <box size="0.1 0.1 0.1" />
-      </geometry>
-      <material name="Cyan">
-        <color rgba="0 1.0 1.0 1.0"/>
-      </material>
-    </visual>
-    <!-- <collision>
-      <origin xyz="0 0 0" rpy="0 0 0"/>
-      <geometry>
-        <box size="0.1 0.1 0.1" />
-      </geometry>
-    </collision> -->
-  </link>
   <!--left wheelLeg model-->
-  <xacro:macro name="LeftWheelLeg" params="name x y z">
+  <xacro:macro name="LeftWheelLeg" params="name x y z parent">
     <link name="${name}">
       <inertial>
@@ -70,5 +47,5 @@
         rpy="1.5708 -1.5708 3.1416" />
       <parent
-        link="base_link" />
+        link="${parent}" />
       <child
         link="${name}" />
@@ -183,5 +160,5 @@
   </xacro:macro>
   <!--right wheelLeg model-->
-  <xacro:macro name="RightWheelLeg" params="name x y z">
+  <xacro:macro name="RightWheelLeg" params="name x y z parent">
     <link name="${name}">
       <inertial>
@@ -228,5 +205,5 @@
         rpy="1.5708 1.5708 0.0" />
       <parent
-        link="base_link" />
+        link="${parent}" />
       <child
         link="${name}" />

Commit message: setup Rhex Mode

File: wheelleg_description/urdf/Hexapod.xacro (robot description, xacro)
@@ -5,4 +5,5 @@
   <!--load gazebo specific configuration-->
   <xacro:include filename="$(find wheelleg_description)/urdf/WheelLeg.gazebo"/>
+  <xacro:include filename="$(find wheelleg_description)/urdf/imu.xacro"/>
   <!--load control interface for robot-->
   <gazebo>
@@ -14,5 +15,5 @@
   <link name="base_link">
     <inertial>
-      <origin xyz="0.05 0.05 0.05" rpy="0 0 0"/>
+      <origin xyz="0.25 0.150 0.005" rpy="0 0 0"/>
       <mass value="1"/>
       <inertia ixx="0.00167"  ixy="0"  ixz="0" iyy="0.00167" iyz="0" izz="0.00167" />
@@ -21,5 +22,5 @@
       <origin xyz="0 0 0" rpy="0 0 0" />
       <geometry>
-        <box size="0.1 0.1 0.1" />
+        <box size="0.5 0.300 0.01" />
       </geometry>
       <material name="Cyan">
@@ -27,18 +28,60 @@
       </material>
     </visual>
-    <!-- <collision>
-      <origin xyz="0 0 0" rpy="0 0 0"/>
+    <collision>
+      <origin xyz="0.25 0.150 0.01" rpy="0 0 0"/>
       <geometry>
-        <box size="0.1 0.1 0.1" />
+        <box size="0.5 0.300 0.01" />
       </geometry>
-    </collision> -->
+    </collision>
   </link>
+  <joint name="dummy_base" type="fixed">
+    <origin xyz="0 0 0" rpy="0 0 0"/>
+    <parent link="base_link"/>
+    <child link="base_link_decoration"/>
+    <axis xyz="0 0 1"/>
+  </joint>
+  <link name="base_link_decoration">
+    <inertial>
+      <origin xyz="0.05 0.190 0.005" rpy="0 0 0"/>
+      <mass value="1"/>
+      <inertia ixx="0.00167"  ixy="0"  ixz="0" iyy="0.00167" iyz="0" izz="0.00167" />
+    </inertial>
+    <visual>
+      <origin xyz="0 0 0" rpy="0 0 0" />
+      <geometry>
+        <box size="0.1 0.380 0.01" />
+      </geometry>
+      <material name="Cyan">
+        <color rgba="0 1.0 1.0 1.0"/>
+      </material>
+    </visual>
+  </link>
+  <xacro:IMU connected_to="base_link" imu_name="imu" xyz="0. 0. .05" rpy="0. 0. 0."/>
+  <gazebo>
+      <plugin name="imu_controller" filename="libgazebo_ros_imu.so">
+      <alwaysOn>true</alwaysOn>
+      <updateRate>30</updateRate>
+      <bodyName>imu</bodyName>   <!--imu_link -->
+      <topicName>imu/data</topicName>
+      <serviceName>imu/is_calibrated</serviceName>
+      <gaussianNoise>0.1</gaussianNoise>
+      <xyzOffsets>0 0 0</xyzOffsets>
+      <rpyOffsets>0 0 0</rpyOffsets>
+      </plugin>
+  </gazebo>
+  <!--publish robot odom to world-->
   <!--define joints-->
-  <xacro:LeftWheelLeg name="LF" x="0.4" y="0.2" z="0.02" parent="base_link"/>
-  <xacro:LeftWheelLeg name="LM" x="0" y="0.3" z="0.02" parent="base_link"/>
-  <xacro:LeftWheelLeg name="LB" x="-0.4" y="0.2" z="0.02" parent="base_link"/>
-  <xacro:RightWheelLeg name="RF" x="0.4" y="-0.2" z="0.02" parent="base_link"/>
-  <xacro:RightWheelLeg name="RM" x="0" y="-0.3" z="0.02" parent="base_link"/>
-  <xacro:RightWheelLeg name="RB" x="-0.4" y="-0.2" z="0.02" parent="base_link"/>
+  <xacro:LeftWheelLeg name="LF"  x="0.21" y="0.116" z="-0.026" parent="base_link"/>
+  <xacro:joint_box name="LF_Box" x="0.21" y="0.116" z="-0.026" parent="base_link"/>
+  <xacro:LeftWheelLeg name="LM"  x="0" y="0.168" z="-0.026" parent="base_link"/>
+  <xacro:joint_box name="LM_Box" x="0" y="0.168" z="-0.026" parent="base_link"/>
+  <xacro:LeftWheelLeg name="LB"  x="-0.21" y="0.116" z="-0.026" parent="base_link"/>
+  <xacro:joint_box name="LB_Box" x="-0.21" y="0.116" z="-0.026" parent="base_link"/>
+  <xacro:RightWheelLeg name="RF" x="0.21" y="-0.116" z="-0.026" parent="base_link"/>
+  <xacro:joint_box name="RF_Box" x="0.21" y="-0.116" z="-0.026" parent="base_link"/>
+  <xacro:RightWheelLeg name="RM" x="0" y="-0.168" z="-0.026" parent="base_link"/>
+  <xacro:joint_box name="RM_Box" x="0" y="-0.168" z="-0.026" parent="base_link"/>
+  <xacro:RightWheelLeg name="RB" x="-0.21" y="-0.116" z="-0.026" parent="base_link"/>
+  <xacro:joint_box name="RB_Box" x="-0.21" y="-0.116" z="-0.026" parent="base_link"/>
   <!--add gazebo joint configures-->
   <xacro:wheelLegJointConfig name="LF" />

File: wheelleg_description/urdf/WheelLeg.xacro (robot description, xacro)
@@ -1,4 +1,34 @@
 <?xml version="1.0" encoding="utf-8"?>
 <robot xmlns:xacro="http://www.ros.org/wiki/xacro" >
+  <xacro:macro name="joint_box" params="name x y z parent">
+    <joint name="${name}_fixed_joint" type="fixed">
+      <origin xyz="${x} ${y} ${z}" rpy="0 0 0"/>
+      <parent link="${parent}"/>
+      <child link="${name}"/>
+      <axis xyz="0 0 1"/>
+    </joint>
+    <link name="${name}">
+      <inertial>
+        <origin xyz="0.025 0.0375 0.025" rpy="0 0 0"/>
+        <mass value="0.01"/>
+        <inertia ixx="0.000167"  ixy="0"  ixz="0" iyy="0.000167" iyz="0" izz="0.000167" />
+      </inertial>
+      <visual>
+        <origin xyz="0 0 0" rpy="0 0 0" />
+        <geometry>
+          <box size="0.05 0.075 0.05" />
+        </geometry>
+        <material name="Cyan">
+          <color rgba="0 1.0 1.0 1.0"/>
+        </material>
+      </visual>
+      <collision>
+         <origin xyz="0.025 0.0375 0.025" rpy="0 0 0"/>
+        <geometry>
+          <box size="0.05 0.075 0.05" />
+        </geometry>
+      </collision>
+    </link>
+  </xacro:macro>
   <!--left wheelLeg model-->
   <xacro:macro name="LeftWheelLeg" params="name x y z parent">

Commit message: locomotion video version

File: wheelleg_description/urdf/Hexapod.xacro (robot description, xacro)
@@ -14,5 +14,5 @@
   <link name="base_link">
     <inertial>
-      <origin xyz="0.05 0.05 0.05" rpy="0 0 0"/>
+      <origin xyz="0 0 0" rpy="0 0 0"/>
       <mass value="1"/>
       <inertia ixx="0.00167"  ixy="0"  ixz="0" iyy="0.00167" iyz="0" izz="0.00167" />
@@ -21,5 +21,5 @@
       <origin xyz="0 0 0" rpy="0 0 0" />
       <geometry>
-        <box size="0.1 0.1 0.1" />
+        <box size="0.5 0.300 0.01" />
       </geometry>
       <material name="Cyan">
@@ -27,18 +27,46 @@
       </material>
     </visual>
-    <!-- <collision>
+    <collision>
       <origin xyz="0 0 0" rpy="0 0 0"/>
       <geometry>
-        <box size="0.1 0.1 0.1" />
+        <box size="0.5 0.300 0.01" />
       </geometry>
-    </collision> -->
+    </collision>
+  </link>
+  <joint name="dummy_base" type="fixed">
+    <origin xyz="0 0 0" rpy="0 0 0"/>
+    <parent link="base_link"/>
+    <child link="base_link_decoration"/>
+    <axis xyz="0 0 1"/>
+  </joint>
+  <link name="base_link_decoration">
+    <inertial>
+      <origin xyz="0.05 0.190 0.005" rpy="0 0 0"/>
+      <mass value="1"/>
+      <inertia ixx="0.00167"  ixy="0"  ixz="0" iyy="0.00167" iyz="0" izz="0.00167" />
+    </inertial>
+    <visual>
+      <origin xyz="0 0 0" rpy="0 0 0" />
+      <geometry>
+        <box size="0.1 0.380 0.01" />
+      </geometry>
+      <material name="Cyan">
+        <color rgba="0 1.0 1.0 1.0"/>
+      </material>
+    </visual>
   </link>
   <!--define joints-->
-  <xacro:LeftWheelLeg name="LF" x="0.4" y="0.2" z="0.02" parent="base_link"/>
-  <xacro:LeftWheelLeg name="LM" x="0" y="0.3" z="0.02" parent="base_link"/>
-  <xacro:LeftWheelLeg name="LB" x="-0.4" y="0.2" z="0.02" parent="base_link"/>
-  <xacro:RightWheelLeg name="RF" x="0.4" y="-0.2" z="0.02" parent="base_link"/>
-  <xacro:RightWheelLeg name="RM" x="0" y="-0.3" z="0.02" parent="base_link"/>
-  <xacro:RightWheelLeg name="RB" x="-0.4" y="-0.2" z="0.02" parent="base_link"/>
+  <xacro:LeftWheelLeg name="LF"  x="0.21" y="0.116" z="-0.026" parent="base_link"/>
+  <xacro:joint_box name="LF_Box" x="0.21" y="0.116" z="-0.026" parent="base_link"/>
+  <xacro:LeftWheelLeg name="LM"  x="0" y="0.168" z="-0.026" parent="base_link"/>
+  <xacro:joint_box name="LM_Box" x="0" y="0.168" z="-0.026" parent="base_link"/>
+  <xacro:LeftWheelLeg name="LB"  x="-0.21" y="0.116" z="-0.026" parent="base_link"/>
+  <xacro:joint_box name="LB_Box" x="-0.21" y="0.116" z="-0.026" parent="base_link"/>
+  <xacro:RightWheelLeg name="RF" x="0.21" y="-0.116" z="-0.026" parent="base_link"/>
+  <xacro:joint_box name="RF_Box" x="0.21" y="-0.116" z="-0.026" parent="base_link"/>
+  <xacro:RightWheelLeg name="RM" x="0" y="-0.168" z="-0.026" parent="base_link"/>
+  <xacro:joint_box name="RM_Box" x="0" y="-0.168" z="-0.026" parent="base_link"/>
+  <xacro:RightWheelLeg name="RB" x="-0.21" y="-0.116" z="-0.026" parent="base_link"/>
+  <xacro:joint_box name="RB_Box" x="-0.21" y="-0.116" z="-0.026" parent="base_link"/>
   <!--add gazebo joint configures-->
   <xacro:wheelLegJointConfig name="LF" />

File: wheelleg_description/urdf/Quadraped.xacro (robot description, xacro)
@@ -12,7 +12,8 @@
   </gazebo>
    <!--define robot base link-->
+   <!--define robot base link-->
   <link name="base_link">
     <inertial>
-      <origin xyz="0.05 0.05 0.05" rpy="0 0 0"/>
+      <origin xyz="0 0 0" rpy="0 0 0"/>
       <mass value="1"/>
       <inertia ixx="0.00167"  ixy="0"  ixz="0" iyy="0.00167" iyz="0" izz="0.00167" />
@@ -21,5 +22,5 @@
       <origin xyz="0 0 0" rpy="0 0 0" />
       <geometry>
-        <box size="0.1 0.1 0.1" />
+        <box size="0.5 0.300 0.01" />
       </geometry>
       <material name="Cyan">
@@ -27,16 +28,19 @@
       </material>
     </visual>
-    <!-- <collision>
+    <collision>
       <origin xyz="0 0 0" rpy="0 0 0"/>
       <geometry>
-        <box size="0.1 0.1 0.1" />
+        <box size="0.5 0.300 0.01" />
       </geometry>
-    </collision> -->
+    </collision>
   </link>
-  <!--define joints-->
-  <xacro:LeftWheelLeg name="LF" x="0.4" y="0.2" z="0.02" parent="base_link" />
-  <xacro:LeftWheelLeg name="LB" x="-0.4" y="0.2" z="0.02" parent="base_link"/>
-  <xacro:RightWheelLeg name="RF" x="0.4" y="-0.2" z="0.02" parent="base_link"/>
-  <xacro:RightWheelLeg name="RB" x="-0.4" y="-0.2" z="0.02" parent="base_link"/>
+  <xacro:LeftWheelLeg name="LF"  x="0.21" y="0.116" z="-0.026" parent="base_link"/>
+  <xacro:joint_box name="LF_Box" x="0.21" y="0.116" z="-0.026" parent="base_link"/>
+  <xacro:LeftWheelLeg name="LB"  x="-0.21" y="0.116" z="-0.026" parent="base_link"/>
+  <xacro:joint_box name="LB_Box" x="-0.21" y="0.116" z="-0.026" parent="base_link"/>
+  <xacro:RightWheelLeg name="RF" x="0.21" y="-0.116" z="-0.026" parent="base_link"/>
+  <xacro:joint_box name="RF_Box" x="0.21" y="-0.116" z="-0.026" parent="base_link"/>
+  <xacro:RightWheelLeg name="RB" x="-0.21" y="-0.116" z="-0.026" parent="base_link"/>
+  <xacro:joint_box name="RB_Box" x="-0.21" y="-0.116" z="-0.026" parent="base_link"/>
   <!--add gazebo joint configures-->
   <xacro:wheelLegJointConfig name="LF" />

File: wheelleg_description/urdf/WheelLeg.xacro (robot description, xacro)
@@ -1,4 +1,34 @@
 <?xml version="1.0" encoding="utf-8"?>
 <robot xmlns:xacro="http://www.ros.org/wiki/xacro" >
+  <xacro:macro name="joint_box" params="name x y z parent">
+    <joint name="${name}_fixed_joint" type="fixed">
+      <origin xyz="${x} ${y} ${z}" rpy="0 0 0"/>
+      <parent link="${parent}"/>
+      <child link="${name}"/>
+      <axis xyz="0 0 1"/>
+    </joint>
+    <link name="${name}">
+      <inertial>
+        <origin xyz="0.0 0.0 0.0" rpy="0 0 0"/>
+        <mass value="0.01"/>
+        <inertia ixx="0.000167"  ixy="0"  ixz="0" iyy="0.000167" iyz="0" izz="0.000167" />
+      </inertial>
+      <visual>
+        <origin xyz="0 0 0" rpy="0 0 0" />
+        <geometry>
+          <box size="0.05 0.075 0.05" />
+        </geometry>
+        <material name="Cyan">
+          <color rgba="0 1.0 1.0 1.0"/>
+        </material>
+      </visual>
+      <!-- <collision>
+         <origin xyz="0.0 0.0 0.0" rpy="0 0 0"/>
+        <geometry>
+          <box size="0.05 0.075 0.05" />
+        </geometry>
+      </collision> -->
+    </link>
+  </xacro:macro>
   <!--left wheelLeg model-->
   <xacro:macro name="LeftWheelLeg" params="name x y z parent">
