Commit message: added playground

File: stairs_playground/urdf/stairs_base.xacro (robot description, xacro)
@@ -28,16 +28,11 @@
         </link>
         <xacro:if value="${stairs-1}">
-            <xacro:stairs stairs="${stairs-1}" xpos="0" ypos="${ypos+stair_length/2}" zpos="${zpos+stair_height/2}" stair_length="${stair_length}" stair_width="${stair_width}" stair_height="${stair_height}"/>
+            <xacro:stairs stairs="${stairs-1}" xpos="${stair_width/2}" ypos="${ypos+stair_length}" zpos="${zpos+stair_height/2}" stair_length="${stair_length}" stair_width="${stair_width}" stair_height="${stair_height}"/>
         </xacro:if>
     </xacro:macro>
-    <xacro:macro name="group_of_stairs" params="num stair_length stair_width stair_height">
+    <xacro:macro name="group_of_stairs" params="num stair_width stair_length stair_height">
         <!--dummy base link-->
         <link name="base_link"/>
-        <xacro:stairs stairs="${num}" xpos="0" ypos="0" zpos="${stair_height/2}" stair_length="${stair_length}" stair_width="${stair_width}" stair_height="${stair_height}"/>
-    </xacro:macro>
-    <xacro:macro name="single_stair" params="stair_length stair_width stair_height">
-        <!--dummy base link-->
-        <link name="base_link"/>
-        <xacro:stairs stairs="1" xpos="0" ypos="0" zpos="${stair_height/2}" stair_length="${stair_length}" stair_width="${stair_width}" stair_height="${stair_height}"/>
+        <xacro:stairs stairs="${num}" xpos="${stair_width/2}" ypos="${stair_length/2}" zpos="${stair_height/2}" stair_length="${stair_length}" stair_width="${stair_width}" stair_height="${stair_height}"/>
     </xacro:macro>
 </robot>

File: wheelleg_gazebo/world/urdf/test.xacro (robot description, xacro)
@@ -1,7 +1,7 @@
 <?xml version="1.0" encoding="utf-8"?>
 <robot xmlns:xacro="http://www.ros.org/wiki/xacro"  name="aaa">
-  <link name="base_link">
-  </link>
   <xacro:include filename="$(find wheelleg_gazebo)/world/urdf/stairs.xacro"/>
-  <xacro:group_of_stairs num="5" xpos="0" ypos="0" zpos="0"/>
+<!--
+  <xacro:group_of_stairs num="20" stair_length="2" stair_width="1" stair_height="0.2"/> -->
+  <xacro:single_stair stair_length="1" stair_width="2" stair_height="0.2"/>
 </robot>

Commit message: modified hexapod gait policy

File: stairs_playground/urdf/stairs_base.xacro (robot description, xacro)
@@ -3,5 +3,5 @@
     <xacro:macro name="stairs" params="stairs xpos ypos zpos stair_length stair_width stair_height">
         <joint name="stair_joint_origin_${stairs}" type="fixed">
-            <origin rpy="0 0 0" xyz="0 0 0"/>
+            <origin rpy="0 0 -1.570795" xyz="0 0 0"/>
             <parent link="base_link"/>
             <child link="stair_link_${stairs}"/>

File: wheelleg_description/urdf/Segway.xacro (robot description, xacro)
@@ -38,5 +38,5 @@
     <child link="z_dummy_link"/>
     <limit effort="30" velocity="100.0" lower="-200" upper="200" />
-    <axis xyz="0 0 1"/>\
+    <axis xyz="0 0 1"/>
   </joint>
   <link name="z_dummy_link">

Commit message: Simulation modified for robio final submission.

File: stairs_playground/urdf/stairs_base.xacro (robot description, xacro)
@@ -27,4 +27,9 @@
             </inertial>
         </link>
+        <gazebo reference="stair_link_${stairs}">
+            <material>Gazebo/Red</material>
+            <mu1>0.001</mu1>
+            <mu2>0.001</mu2>
+        </gazebo>
         <xacro:if value="${stairs-1}">
             <xacro:stairs stairs="${stairs-1}" xpos="${stair_width/2}" ypos="${ypos+stair_length}" zpos="${zpos+stair_height/2}" stair_length="${stair_length}" stair_width="${stair_width}" stair_height="${stair_height}"/>

File: wheelleg_description/urdf/Hexapod.xacro (robot description, xacro)
@@ -15,5 +15,5 @@
   <link name="base_link">
     <inertial>
-      <origin xyz="0.25 0.150 0.005" rpy="0 0 0"/>
+      <origin xyz="0 0 0" rpy="0 0 0"/>
       <mass value="1"/>
       <inertia ixx="0.00167"  ixy="0"  ixz="0" iyy="0.00167" iyz="0" izz="0.00167" />
@@ -29,5 +29,5 @@
     </visual>
     <collision>
-      <origin xyz="0.25 0.150 0.01" rpy="0 0 0"/>
+      <origin xyz="0 0 0" rpy="0 0 0"/>
       <geometry>
         <box size="0.5 0.300 0.01" />
@@ -57,10 +57,9 @@
     </visual>
   </link>
-  <xacro:IMU connected_to="base_link" imu_name="imu" xyz="0. 0. .05" rpy="0. 0. 0."/>
   <gazebo>
       <plugin name="imu_controller" filename="libgazebo_ros_imu.so">
       <alwaysOn>true</alwaysOn>
       <updateRate>30</updateRate>
-      <bodyName>imu</bodyName>   <!--imu_link -->
+      <bodyName>base_link</bodyName>   <!--imu_link -->
       <topicName>imu/data</topicName>
       <serviceName>imu/is_calibrated</serviceName>

File: wheelleg_description/urdf/WheelLeg.xacro (robot description, xacro)
@@ -10,5 +10,5 @@
     <link name="${name}">
       <inertial>
-        <origin xyz="0.025 0.0375 0.025" rpy="0 0 0"/>
+        <origin xyz="0.0 0.0 0.0" rpy="0 0 0"/>
         <mass value="0.01"/>
         <inertia ixx="0.000167"  ixy="0"  ixz="0" iyy="0.000167" iyz="0" izz="0.000167" />
@@ -23,10 +23,10 @@
         </material>
       </visual>
-      <collision>
-         <origin xyz="0.025 0.0375 0.025" rpy="0 0 0"/>
+      <!-- <collision>
+         <origin xyz="0.0 0.0 0.0" rpy="0 0 0"/>
         <geometry>
           <box size="0.05 0.075 0.05" />
         </geometry>
-      </collision>
+      </collision> -->
     </link>
   </xacro:macro>
@@ -123,8 +123,8 @@
       </collision>
     </link>
-    <joint name="${name}RA_Joint" type="continuous">
+    <joint name="${name}RA_Joint" type="fixed">
       <origin
         xyz="0 -0.08 0.038242"
-        rpy="3.1416 0 1.5708" />
+        rpy="3.1416 0 2.0708" />
       <parent
         link="${name}" />
@@ -175,5 +175,5 @@
       </collision>
     </link>
-    <joint name="${name}RB_Joint" type="continuous">
+    <joint name="${name}RB_Joint" type="fixed">
       <origin
         xyz="0 0.08 0.038242"
@@ -281,8 +281,8 @@
       </collision>
     </link>
-    <joint name="${name}RA_Joint" type="continuous">
+    <joint name="${name}RA_Joint" type="fixed">
       <origin
         xyz="0 -0.08 0.038244"
-        rpy="0 0 1.5708" />
+        rpy="0 0 1.0708" />
       <parent
         link="${name}" />
@@ -333,5 +333,5 @@
       </collision>
     </link>
-    <joint name="${name}RB_Joint" type="continuous">
+    <joint name="${name}RB_Joint" type="fixed">
       <origin
         xyz="0 0.08 0.038244"

Commit message: Recording LegReverse Mode

File: stairs_playground/urdf/stairs_base.xacro (robot description, xacro)
@@ -28,7 +28,6 @@
         </link>
         <gazebo reference="stair_link_${stairs}">
-            <material>Gazebo/Red</material>
-            <mu1>0.001</mu1>
-            <mu2>0.001</mu2>
+            <mu1>0.1</mu1>
+            <mu2>0.1</mu2>
         </gazebo>
         <xacro:if value="${stairs-1}">

File: wheelleg_description/urdf/Segway.xacro (robot description, xacro)
@@ -34,5 +34,5 @@
   </gazebo>
   <joint name="z_dof" type="prismatic">
-    <origin xyz="0 0 0" rpy="0 0 0"/>
+    <origin xyz="0 0 0" rpy="0 0 3.1415926"/>
     <parent link="static_base"/>
     <child link="z_dummy_link"/>
@@ -86,4 +86,17 @@
     </collision> -->
   </link>
+  <joint name="camera_joint" type="fixed">
+    <origin xyz="0 0.7 0" rpy="0 0 -1.570796326794897"/>
+    <parent link="base_link"/>
+    <child link="camera_link"/>
+    <axis xyz="0 0 1"/>
+  </joint>
+  <link name="camera_link">
+    <inertial>
+      <origin xyz="0.05 0.05 0.05" rpy="0 0 0"/>
+      <mass value="0.001"/>
+      <inertia ixx="0.000167"  ixy="0"  ixz="0" iyy="0.000167" iyz="0" izz="0.000167" />
+    </inertial>
+  </link>
   <!--define joints-->
   <xacro:LeftWheelLeg name="L" x="0" y="0.2" z="0.0" parent="base_link"/>
